File: ECPR_EMITTER.sch (EAGLE design)
At the start: 22 parts, among them IC1 78L05, IC2 ATMEGA8-PU, J1 0802_SCREEN, Q1 BFR96, U1 AD9850 DDS Module

Commit message: FUCK
Changed lines of the file:
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@@
 </classes>
 <parts>
-<part name="Q1" library="transistor-small-signal" library_urn="urn:adsk.eagle:library:401" deviceset="BFR96" device="" package3d_urn="urn:adsk.eagle:package:28760/1"/>
+<part name="Q1" library="transistor-small-signal" deviceset="BFR96" device=""/>
 <part name="GND1" library="supply" deviceset="GND" device=""/>
 <part name="GND2" library="supply" deviceset="GND" device=""/>
@@
 <part name="U$1" library="computronics.com.au" deviceset="ANTENNA" device="" value="ANT."/>
 <part name="L1" library="inductors" deviceset="82114R" device=""/>
-<part name="C3" library="capacitor-wima" library_urn="urn:adsk.eagle:library:116" deviceset="C" device="5/3" package3d_urn="urn:adsk.eagle:package:5433/1" value="1nF"/>
+<part name="C3" library="capacitor-wima" deviceset="C" device="5/3" value="1nF"/>
 <part name="V1" library="supply0" deviceset="VBAT" device=""/>
 <part name="V2" library="supply0" deviceset="VBAT" device=""/>
@@
 <part name="U1" library="dds-module-ad9850" deviceset="DDS_MODULE:AD9850" device="DDS_MODULE" value="AD9850 DDS Module"/>
 <part name="P+5" library="supply1" deviceset="VCC" device=""/>
-<part name="SUPPLY1" library="supply2" library_urn="urn:adsk.eagle:library:372" deviceset="GND" device=""/>
+<part name="SUPPLY1" library="supply2" deviceset="GND" device=""/>
 <part name="FRAME1" library="SparkFun-Aesthetics" deviceset="FRAME-LETTER" device="NO_PACKAGE"/>
 <part name="GND7" library="supply0" deviceset="GND" device=""/>
@@
 which will not be processed correctly with this version.
 </note>
-<note version="8.2" severity="warning">
-Since Version 8.2, EAGLE supports online libraries. The ids
-of those online libraries will not be understood (or retained)
-with this version.
-</note>
-<note version="8.3" severity="warning">
-Since Version 8.3, EAGLE supports URNs for individual library
-assets (packages, symbols, and devices). The URNs of those assets
-will not be understood (or retained) with this version.
-</note>
-<note version="8.3" severity="warning">
-Since Version 8.3, EAGLE supports the association of 3D packages
-with devices in libraries, schematics, and board files. Those 3D
-packages will not be understood (or retained) with this version.
-</note>
 </compatibility>
